Commit message: coorected map to odom transformation based on camera data

File: model/cassiopeia.urdf (robot description, URDF)
Before this commit: robot space_robot, 7 links, 6 joints
Joints:
- joint left_shoulder: origin xyz=0.15 -0.1 0.1 rpy=0 0 0 -> xyz=0.15 0.1 0.1 rpy=0 0 0
- joint right_shoulder: origin xyz=0.15 0.1 0.1 rpy=0 0 0 -> xyz=0.15 -0.1 0.1 rpy=0 0 0

Commit message: implement hardware interface for controlling all joints

File: model/cassiopeia.urdf (robot description, URDF)
Before this commit: robot space_robot, 7 links, 6 joints
Joints:
- joint left_shoulder: limit lower=-2.57 upper=1.57 effort=1 velocity=0.5 -> lower=-0.57 upper=0.57 effort=1 velocity=0.5

Commit message: lot of stuff

File: model/cassiopeia.urdf (robot description, URDF)
Before this commit: robot space_robot, 7 links, 6 joints
Links:
- added link T1, mass 1; visual cylinder length=0.05 radius=0.01
- added link T2, mass 1; visual cylinder length=0.05 radius=0.01
- added link T3, mass 1; visual cylinder length=0.05 radius=0.01
- added link front_mouse, mass 15; visual box size=0.12 .07 .03
- added link left_mouse, mass 15; visual box size=0.12 .07 .03
- added link reaction_wheel; visual box size=0.1 0.1 .03
- added link right_mouse, mass 15; visual box size=0.12 .07 .03
- link base_link: mass 15 -> None; geometry visual cylinder length=0.37 radius=0.15
Joints:
- added joint f_odom: type fixed, parent base_link, child front_mouse, origin xyz=0.15 0 0 rpy=0 0 0
- added joint j_T1: type fixed, parent base_link, child T1, origin xyz=0.085 0.147224319 0.23 rpy=0 0 -0.52
- added joint j_T2: type fixed, parent base_link, child T2, origin xyz=-0.17 0 0.23 rpy=0 0 1.57
- added joint j_T3: type fixed, parent base_link, child T3, origin xyz=0.085 -0.147224319 0.23 rpy=0 0 -2.62
- added joint l_odom: type fixed, parent base_link, child left_mouse, origin xyz=-0.1 0.1 0 rpy=0 0 0
- added joint r_odom: type fixed, parent base_link, child right_mouse, origin xyz=-0.1 -0.1 0 rpy=0 0 0
- added joint reaction_wheel_joint: type revolute, parent base_link, child reaction_wheel, origin xyz=0 0 0 rpy=0 0 0, axis 0 0 1, limit lower=-10.57 upper=20.57 effort=10 velocity=200.5
- joint left_wrist: type revolute -> fixed
- joint right_wrist: type revolute -> fixed
